File: teensy_to_autodriver.sch (KiCad schematic (older format))
At the start: 7 parts, among them J1 PIN_ARRAY_5X2, J2 PIN_ARRAY_3X2, J3 PIN_ARRAY_2X1, J4 PIN_ARRAY_2X1, J5 PIN_ARRAY_2X1, J6 PIN_ARRAY_2X1, U1 TEENSY3.1

Commit message: Created version 0.2 of design. Added header for angle sensor.
Parts:
- added J7: PIN_ARRAY_3X1, HEADER_3X1:HEADER_3X1, symbol PIN_ARRAY_3X1
Connections:
- net GND: now also J7.1 (Pin_1)
- net A1: now reaches U1.22 (D15,A1,TOUCH)
- net A1: now also J7.3 (Pin_3)
- net 3V3: now reaches U1.31 (3V3)
- net 3V3: now also J7.2 (Pin_2)
- no-connect marks 42 -> 45
Other:
- note added: "Angle Sensor"
Changed lines of the file:
@@
 LIBS:pin_array_2x1
 LIBS:teensy3
+LIBS:pin_array_3x1
 LIBS:teensy_to_autodriver-cache
 EELAYER 25 0
@@
 L PWR_FLAG #FLG07
 U 1 1 5A568096
-P 10150 1500
-F 0 "#FLG07" H 10150 1575 50  0001 C CNN
-F 1 "PWR_FLAG" H 10150 1650 50  0000 C CNN
-F 2 "" H 10150 1500 50  0001 C CNN
-F 3 "" H 10150 1500 50  0001 C CNN
-	1    10150 1500
-	1    0    0    -1
-$EndComp
-Wire Wire Line
-	10150 1500 10150 1600
-Wire Wire Line
-	10150 1600 10000 1600
-Text Label 10000 1600 2    60   ~ 0
+P 10650 1850
+F 0 "#FLG07" H 10650 1925 50  0001 C CNN
+F 1 "PWR_FLAG" H 10650 2000 50  0000 C CNN
+F 2 "" H 10650 1850 50  0001 C CNN
+F 3 "" H 10650 1850 50  0001 C CNN
+	1    10650 1850
+	1    0    0    -1
+$EndComp
+Wire Wire Line
+	10650 1850 10650 1950
+Wire Wire Line
+	10650 1950 10500 1950
+Text Label 10500 1950 2    60   ~ 0
 +5V
 $Comp
 L PWR_FLAG #FLG08
 U 1 1 5A5683BF
-P 10600 1500
-F 0 "#FLG08" H 10600 1575 50  0001 C CNN
-F 1 "PWR_FLAG" H 10600 1650 50  0000 C CNN
-F 2 "" H 10600 1500 50  0001 C CNN
-F 3 "" H 10600 1500 50  0001 C CNN
-	1    10600 1500
-	1    0    0    -1
-$EndComp
-Wire Wire Line
-	10600 1500 10600 1650
+P 10650 2300
+F 0 "#FLG08" H 10650 2375 50  0001 C CNN
+F 1 "PWR_FLAG" H 10650 2450 50  0000 C CNN
+F 2 "" H 10650 2300 50  0001 C CNN
+F 3 "" H 10650 2300 50  0001 C CNN
+	1    10650 2300
+	1    0    0    -1
+$EndComp
+Wire Wire Line
+	10650 2300 10650 2450
 $Comp
 L GND #PWR09
 U 1 1 5A568415
-P 10600 1650
-F 0 "#PWR09" H 10600 1400 50  0001 C CNN
-F 1 "GND" H 10600 1500 50  0000 C CNN
-F 2 "" H 10600 1650 50  0001 C CNN
-F 3 "" H 10600 1650 50  0001 C CNN
-	1    10600 1650
+P 10650 2450
+F 0 "#PWR09" H 10650 2200 50  0001 C CNN
+F 1 "GND" H 10650 2300 50  0000 C CNN
+F 2 "" H 10650 2450 50  0001 C CNN
+F 3 "" H 10650 2450 50  0001 C CNN
+	1    10650 2450
 	1    0    0    -1
 $EndComp
@@
 Text Label 4050 1250 0    60   ~ 0
 DAC
+$Comp
+L PIN_ARRAY_3X1 J7
+U 1 1 5A5F9B3F
+P 8250 3300
+F 0 "J7" H 8250 3500 50  0000 C CNN
+F 1 "PIN_ARRAY_3X1" H 8250 3100 50  0000 C CNN
+F 2 "HEADER_3X1:HEADER_3X1" H 8250 3300 50  0001 C CNN
+F 3 "" H 8250 3300 50  0001 C CNN
+	1    8250 3300
+	1    0    0    -1
+$EndComp
+Text Notes 7950 3750 0    60   ~ 0
+Angle Sensor
+Wire Wire Line
+	8050 3200 7850 3200
+Wire Wire Line
+	8050 3300 7850 3300
+Wire Wire Line
+	8050 3400 7850 3400
+Wire Wire Line
+	1800 3750 1600 3750
+Text Label 1600 3750 2    60   ~ 0
+3V3
+Text Label 7850 3300 2    60   ~ 0
+3V3
+Text Label 7850 3200 2    60   ~ 0
+GND
+NoConn ~ 1800 3450
+NoConn ~ 1800 3550
+NoConn ~ 1800 3650
+Wire Wire Line
+	1800 2850 1600 2850
 NoConn ~ 1800 2950
-NoConn ~ 1800 2850
+Text Label 1600 2850 2    60   ~ 0
+A1
+Text Label 7850 3400 2    60   ~ 0
+A1
+NoConn ~ 1800 3850
 $EndSCHEMATC
